Commit message: Add simulated realsense to franka.
Signed-off-by: Jelmer de Wolde <jelmer.de.wolde@alliander.com>

File: rcdt_franka/urdf/franka.urdf.xacro (robot description, xacro)
@@ -15,8 +15,5 @@
   <xacro:arg name="robot_ip" default="" />
   <!-- Realsense related: -->
-  <xacro:arg name="load_realsense" default="true" />
-  <xacro:arg name="pos_realsense" default="0.05 0 0.05" />
-  <xacro:arg name="parent_realsense" default="fr3_hand" />
-  <xacro:arg name="rot_realsense" default="0 ${-0.5*pi} 0" />
+  <xacro:arg name="load_realsense" default="false" />
   <!-- Load arm: -->
   <xacro:include filename="$(find franka_description)/robots/common/franka_robot.xacro" />
@@ -41,8 +38,15 @@
   <!-- Load realsense: -->
   <xacro:if value="$(arg load_realsense)">
-    <xacro:include filename="$(find realsense2_description)/urdf/_d435.urdf.xacro" />
-    <xacro:sensor_d435 parent="$(arg parent_realsense)">
-      <origin xyz="$(arg pos_realsense)" rpy="$(arg rot_realsense)" />
-    </xacro:sensor_d435>
+    <xacro:include filename="$(find rcdt_utilities)/urdf/rcdt_realsense_d435.urdf.xacro" />
+    <link name="realsense_link" />
+    <joint name="realsense_link_joint" type="fixed">
+      <origin xyz="0.02 0 0.05" rpy="0 ${-0.5*pi} ${pi}" />
+      <parent link="fr3_hand" />
+      <child link="realsense_link" />
+    </joint>
+    <xacro:rcdt_realsense_d435
+      parent="realsense_link"
+      gazebo="$(arg gazebo)"
+    />
   </xacro:if>
 </robot>
